Commit message: Weekly CodeRelease
Co-authored-by: Aishkrish18 <aishu2.k@gmail.com>
Co-authored-by: Bennett Wetters <contact@bendo.org>
Co-authored-by: Darshana Sanjeewan Adikari <darshanaads@gmail.com>
Co-authored-by: Hendrik <git@h3ndrk.de>
Co-authored-by: Jonathan Hellwig <jonathan.hellwig@posteo.de>
Co-authored-by: Konrad Mösch <konrad@moesch.org>
Co-authored-by: Konrad Nölle <konrad@familie-noelle.de>
Co-authored-by: Maximilian Schmidt <maximilian@schmidt.so>
Co-authored-by: Nicolas Riebesel <nicolas.riebesel@gmx.com>
Co-authored-by: PasGl <pascalgleske+github@gmail.com>
Co-authored-by: alexschirr <alexschirr@gmail.com>
Co-authored-by: andreeja <andrea.essig@tuhh.de>
Co-authored-by: knoellle <konrad@familie-noelle.de>
Co-authored-by: schluis <luis.scheuch@posteo.de>

File: webots/protos/NAO.urdf (robot description, URDF)
Before this commit: robot NAOH25V60, 131 links, 130 joints
Links:
- added link LFoot/Sole
- added link RFoot/Sole
Joints:
- added joint LFoot/Sole_fixedjoint: type fixed, parent LAnkleRoll_link, child LFoot/Sole, origin xyz=-0.04519 0.0 0.0 rpy=0 -1.5708 3.14159, axis 0 0 0
- added joint RFoot/Sole_fixedjoint: type fixed, parent RAnkleRoll_link, child RFoot/Sole, origin xyz=-0.04519 0.0 0.0 rpy=0 -1.5708 3.14159, axis 0 0 0
